Commit message: urdf chang

File: urdf/car1.urdf (robot description, URDF)
Before this commit: robot car1, 10 links, 9 joints
Joints:
- joint dummy_joint: origin (none) -> xyz=0 0 1.428 rpy=0 0 0
- joint jiont1-1: limit lower=-3.14 upper=3.14 effort=100 velocity=1 -> lower=0 upper=0 effort=100 velocity=1; type revolute -> continuous
- joint joint2-1: limit lower=-3.14 upper=3.14 effort=100 velocity=1 -> lower=0 upper=0 effort=100 velocity=1; type revolute -> continuous
- joint joint3-1: limit lower=-3.14 upper=3.14 effort=100 velocity=1 -> lower=0 upper=0 effort=100 velocity=1; type revolute -> continuous
- joint joint4-1: limit lower=-3.14 upper=3.14 effort=100 velocity=1 -> lower=0 upper=0 effort=100 velocity=1; type revolute -> continuous
